Commit message: delet unnessary package, and  fixed issues after upgrade some humble packages.

File: src/gluon_py/urdf/gluon.urdf (robot description, URDF)
Before this commit: robot gluon, 8 links, 7 joints
Joints:
- joint axis_joint_1: limit lower=-2.79 upper=2.79 effort=30 velocity=3.14 -> lower=-2.44 upper=2.44 effort=30 velocity=3.14
- joint axis_joint_2: limit lower=-1.54 upper=1.54 effort=30 velocity=3.14 -> lower=-1.57 upper=1.57 effort=30 velocity=3.14
- joint axis_joint_3: limit lower=-2.79 upper=2.79 effort=30 velocity=3.14 -> lower=-2.44 upper=2.44 effort=30 velocity=3.14
- joint axis_joint_4: limit lower=-2.79 upper=2.79 effort=30 velocity=3.14 -> lower=-2.44 upper=2.44 effort=30 velocity=3.14
- joint axis_joint_5: limit lower=-2.79 upper=2.79 effort=30 velocity=3.14 -> lower=-1.22 upper=3.66 effort=30 velocity=3.14
- joint axis_joint_6: limit lower=-2.79 upper=2.79 effort=30 velocity=3.14 -> lower=-22.16 upper=22.16 effort=30 velocity=3.14
